File: plusle/plusle.kicad_sch (KiCad schematic)
At the start: 7 parts, among them J1 Battery, J2 MotorA, J3 MotorB, SW1 SW_SPST, U1 ESP32-DEVKIT-V1, U2 ROB-14450

Commit message: updated
updated layout and schematic for hive bot (powered by 9v battery with switch)
Parts:
- removed SW1: SW_SPST, Button_Switch_THT:SW_AS11CP, symbol Switch:SW_SPST
- J1, J2, J3: footprint TerminalBlock:TerminalBlock_Altech_AK300-2_P5.00mm -> TerminalBlock:TerminalBlock_Xinya_XY308-2.54-2P_1x02_P2.54mm_Horizontal
Connections:
- net +12V: now also J1.2 (Pin_2)
Changed lines of the file:
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@@
-	(wire
-		(pts
-			(xy 83.82 35.56) (xy 87.63 35.56)
-		)
-		(stroke
-			(width 0)
-			(type default)
-		)
-	)
 	(wire
 		(pts
@@
 	(wire
 		(pts
+			(xy 91.44 35.56) (xy 91.44 30.48)
+		)
+		(stroke
+			(width 0)
+			(type default)
+		)
+	)
+	(wire
+		(pts
 			(xy 63.5 71.12) (xy 57.15 71.12)
 		)
@@
 	(wire
 		(pts
-			(xy 97.79 35.56) (xy 100.33 35.56)
-		)
-		(stroke
-			(width 0)
-			(type default)
-		)
-	)
-	(wire
-		(pts
 			(xy 57.15 118.11) (xy 62.23 118.11)
 		)
@@
 	(wire
 		(pts
-			(xy 83.82 30.48) (xy 83.82 35.56)
-		)
-		(stroke
-			(width 0)
-			(type default)
-		)
-	)
-	(wire
-		(pts
 			(xy 57.15 110.49) (xy 62.23 110.49)
 		)
@@
 		(pts
 			(xy 120.65 81.28) (xy 120.65 85.09)
+		)
+		(stroke
+			(width 0)
+			(type default)
+		)
+	)
+	(wire
+		(pts
+			(xy 100.33 35.56) (xy 91.44 35.56)
 		)
 		(stroke
@@
 	(symbol
 		(lib_id "power:+12V")
-		(at 83.82 30.48 0)
+		(at 91.44 30.48 0)
 		(unit 1)
 		(exclude_from_sim no)
@@
 		(fields_autoplaced yes)
 		(property "Reference" "#PWR03"
-			(at 83.82 34.29 0)
+			(at 91.44 34.29 0)
 			(effects
 				(font
@@
 		)
 		(property "Value" "+12V"
-			(at 83.82 25.4 0)
+			(at 91.44 25.4 0)
 			(effects
 				(font
@@
 		)
 		(property "Footprint" ""
-			(at 83.82 30.48 0)
+			(at 91.44 30.48 0)
 			(effects
 				(font
@@
 		)
 		(property "Datasheet" ""
-			(at 83.82 30.48 0)
+			(at 91.44 30.48 0)
 			(effects
 				(font
@@
 		)
 		(property "Description" ""
-			(at 83.82 30.48 0)
+			(at 91.44 30.48 0)
 			(effects
 				(font
@@
 			)
 		)
-		(property "Footprint" "TerminalBlock:TerminalBlock_Altech_AK300-2_P5.00mm"
+		(property "Footprint" "TerminalBlock:TerminalBlock_Xinya_XY308-2.54-2P_1x02_P2.54mm_Horizontal"
 			(at 105.41 33.02 0)
 			(effects
@@
 	)
 	(symbol
-		(lib_id "Switch:SW_SPST")
-		(at 92.71 35.56 0)
-		(unit 1)
-		(exclude_from_sim no)
-		(in_bom yes)
-		(on_board yes)
-		(dnp no)
-		(fields_autoplaced yes)
-		(property "Reference" "SW1"
-			(at 92.71 30.2092 0)
-			(effects
-				(font
-					(size 1.27 1.27)
-				)
-			)
-		)
-		(property "Value" "SW_SPST"
-			(at 92.71 32.7461 0)
-			(effects
-				(font
-					(size 1.27 1.27)
-				)
-			)
-		)
-		(property "Footprint" "Button_Switch_THT:SW_AS11CP"
-			(at 92.71 35.56 0)
-			(effects
-				(font
-					(size 1.27 1.27)
-				)
-				(hide yes)
-			)
-		)
-		(property "Datasheet" "~"
-			(at 92.71 35.56 0)
-			(effects
-				(font
-					(size 1.27 1.27)
-				)
-				(hide yes)
-			)
-		)
-		(property "Description" "Single Pole Single Throw (SPST) switch"
-			(at 92.71 35.56 0)
-			(effects
-				(font
-					(size 1.27 1.27)
-				)
-				(hide yes)
-			)
-		)
-		(pin "1"
-		)
-		(pin "3"
-		)
-		(instances
-			(project "plusle"
-				(path "/7b8ee2f4-a696-4f79-b685-0a7bb7795b92"
-					(reference "SW1")
-					(unit 1)
-				)
-			)
-		)
-	)
-	(symbol
 		(lib_id "power:+3.3V")
 		(at 120.65 71.12 0)
@@
 			)
 		)
-		(property "Footprint" "TerminalBlock:TerminalBlock_Altech_AK300-2_P5.00mm"
+		(property "Footprint" "TerminalBlock:TerminalBlock_Xinya_XY308-2.54-2P_1x02_P2.54mm_Horizontal"
 			(at 67.31 110.49 0)
 			(effects
@@
 			)
 		)
-		(property "Footprint" "TerminalBlock:TerminalBlock_Altech_AK300-2_P5.00mm"
+		(property "Footprint" "TerminalBlock:TerminalBlock_Xinya_XY308-2.54-2P_1x02_P2.54mm_Horizontal"
 			(at 67.31 118.11 0)
 			(effects

Commit message: NewIteration
new compact board for personal plusle project, non-hive
Parts:
- removed J1: Battery, TerminalBlock:TerminalBlock_Xinya_XY308-2.54-2P_1x02_P2.54mm_Horizontal, symbol Connector_Generic:Conn_01x02
- removed PS1: TSR_1-2450, TSR_1-2433:CONV_TSR_1-2433, symbol TSR_1-2433:TSR_1-2433
- removed U1: ESP32-DEVKIT-V1, Library:MODULE_ESP32_DEVKIT_V1, symbol ESP32-DEVKIT-V1:ESP32-DEVKIT-V1
- removed U2: ROB-14450, Library:MODULE_ROB-14450, symbol ROB-14450:ROB-14450
- added A1: Arduino_Nano_v3.x, Module:Arduino_Nano, symbol MCU_Module:Arduino_Nano_v3.x
- added C1, C2, C3, C4, C5, C6, C7, C8: 0.1uf, Capacitor_SMD:C_0805_2012Metric_Pad1.18x1.45mm_HandSolder, symbol Device:C
- added D1, D2: GREEN, Capacitor_SMD:C_0603_1608Metric_Pad1.08x0.95mm_HandSolder, symbol Device:LED
- added F1: 15A, Fuse:Fuse_1206_3216Metric_Pad1.42x1.75mm_HandSolder, symbol Device:Fuse
- added H1, H2, H3, H4: MountingHole, MountingHole:MountingHole_2.2mm_M2_ISO7380, symbol Mechanical:MountingHole
- added J1: Receiver Connection2, Connector_PinHeader_2.54mm:PinHeader_1x03_P2.54mm_Vertical, symbol Connector:Conn_01x03_Pin
- added J4: Receiver Connection1, Connector_PinHeader_2.54mm:PinHeader_1x03_P2.54mm_Vertical, symbol Connector:Conn_01x03_Pin
- added J5: Battery, Connector_AMASS:AMASS_XT30PW-M_1x02_P2.50mm_Horizontal, symbol Connector_Generic:Conn_01x02
- added R1, R2: 15k, Resistor_SMD:R_0805_2012Metric_Pad1.20x1.40mm_HandSolder, symbol Device:R_US
- added R3, R4: 600, Diode_SMD:D_0805_2012Metric_Pad1.15x1.40mm_HandSolder, symbol Device:R_US
- added SW1: SW_SPST, Button_Switch_THT:SW_AS11CP, symbol Switch:SW_SPST
- added U3, U4: DRV8871DDA, Package_SO:Texas_HTSOP-8-1EP_3.9x4.9mm_P1.27mm_EP2.95x4.9mm_Mask2.4x3.1mm_ThermalVias, symbol Driver_Motor:DRV8871DDA
Connections:
- net +5V: now also A1.27 (+5V), A1.28 (~{RESET}), A1.3 (~{RESET}), C4.1, C5.1, C6.1, J1.2 (Pin_2), J4.2 (Pin_2), R4.1
- net AIn1: now also A1.14 (D11), U3.3 (IN1)
- net AIn2: now also A1.13 (D10), U3.2 (IN2)
- net BIn1: now also A1.9 (D6), U4.3 (IN1)
- net BIn2: now also A1.8 (D5), U4.2 (IN2)
- net GND: now also A1.29 (GND), A1.4 (GND), C1.2, C2.2, C3.2, C4.2, C5.2, C6.2, C7.1, C8.1, D1.1 (K), D2.1 (K), J1.3 (Pin_3), J4.3 (Pin_3), J5.1 (Pin_1), R1.2, R2.2, U3.1 (GND), U3.7 (GND), U3.9 (GND), U4.1 (GND), U4.7 (GND), U4.9 (GND)
- net at J2.1 (Pin_1): now also U3.8 (OUT2)
- net at J2.2 (Pin_2): now also U3.6 (OUT1)
- net at J3.2 (Pin_2): now also U4.6 (OUT1)
- net at J3.1 (Pin_1): now also U4.8 (OUT2)
- new net: F1.1, SW1.1 (A)
- new net: R2.1, U4.4 (ILIM)
- new net: D1.2 (A), R3.2
- new net: R1.1, U3.4 (ILIM)
- new net: J5.2 (Pin_2), SW1.3 (B)
- new net: D2.2 (A), R4.2
- new net +15V: A1.30 (VIN), C1.1, C2.1, C3.1, C7.2, C8.2, F1.2, R3.1, U3.5 (VM), U4.5 (VM)
- new net RCSignalA: A1.22 (A3), J4.1 (Pin_1)
- new net RCSignalB: A1.23 (A4), J1.1 (Pin_1)
- no-connect marks 0 -> 2
Other:
- note added: "MISC."
- note added: "Motor Driver"
- note added: "Nano"
- note added: "Power & Decoupling"
- note added: "RC"
